File: EPDM.kicad_pcb (KiCad board)
At the start: 2 copper layers, 31.4 x 26.9 mm, 25 parts, among them J1 Conn_01x34_MountingPin, J2 Conn_01x24_MountingPin, J3 Conn_01x09_Female, J4 Conn_01x10, J5 Conn_01x10, Q1 IRLML6344

Commit message: EPDM without adapter part
Parts:
- removed J4: Conn_01x10, Connector_PinHeader_1.27mm:PinHeader_1x10_P1.27mm_Vertical
- removed J5: Conn_01x10, Connector_PinHeader_2.54mm:PinHeader_1x10_P2.54mm_Vertical
Routing:
- net GND: track 47.4 -> 33.0 mm
- net +3V3: track 32.4 -> 18.6 mm
- net /CS1: track 33.3 -> 20.0 mm
- net /EPD_DIN: track 31.2 -> 18.1 mm
- net /EPD_BUSY: track 31.8 -> 19.1 mm
- net /EPD_CLK: track 31.9 -> 19.4 mm
- net /EPD_RST: track 29.6 -> 17.4 mm
- net /EPD_CS: track 29.5 -> 17.5 mm
- net /EPD_DC: track 30.4 -> 18.7 mm
- net Net-(J4-Pad10): track 10.4 -> 0.00 mm
Other:
- board size 31.4 x 26.9 mm -> 17.8 x 23.6 mm
- board text removed: "BUSY"
- board text removed: "CLK"
- board text removed: "CS"
- board text removed: "CS1"
- board text removed: "DC"
- board text removed: "DIN"
- board text removed: "GND"
- board text removed: "RST"
- board text removed: "VCC"
