File: EPDM.kicad_sch (KiCad schematic)
At the start: 25 parts, among them J1 Conn_01x34_MountingPin, J2 Conn_01x24_MountingPin, J3 Conn_01x09_Female, J4 Conn_01x10, J5 Conn_01x10, Q1 IRLML6344

Commit message: Size optimization
Parts:
- C12: footprint Capacitor_SMD:C_0603_1608Metric -> Capacitor_SMD:C_0805_2012Metric
Changed lines of the file:
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@@
   )
   (symbol (lib_id "Device:C") (at 147.32 95.25 0) (unit 1)
-    (in_bom yes) (on_board yes)
+    (in_bom yes) (on_board no)
     (property "Reference" "C7" (id 0) (at 150.241 94.0816 0)
       (effects (font (size 1.27 1.27)) (justify left))
@@
     (property "Reference" "C12" (id 0) (at 214.63 85.09 0))
     (property "Value" "10uF/6V" (id 1) (at 217.17 87.63 0))
-    (property "Footprint" "Capacitor_SMD:C_0603_1608Metric" (id 2) (at 209.8548 82.55 0)
+    (property "Footprint" "Capacitor_SMD:C_0805_2012Metric" (id 2) (at 209.8548 82.55 0)
       (effects (font (size 1.27 1.27)) hide)
     )
@@
     )
     (path "/f14b9c48-b14e-4abd-a69a-d0446c13d922"
-      (reference "C12") (unit 1) (value "10uF/6V") (footprint "Capacitor_SMD:C_0603_1608Metric")
+      (reference "C12") (unit 1) (value "10uF/6V") (footprint "Capacitor_SMD:C_0805_2012Metric")
     )
     (path "/38f52602-301f-4546-becb-9bd2b80145d8"
